Commit message: Add files via upload

File: spider_bot/urdf/spider_bot.urdf (robot description, URDF)
Before this commit: robot spider_bot, 9 links, 8 joints
Links:
- removed link hip1
- removed link hip2
- removed link hip3
- removed link hip4
- removed link leg1
- removed link leg2
- removed link leg3
- removed link leg4
- added link hip1_link, mass 0.020238; collision mesh filename=package://spider_bot/meshes/hip1_link.STL; visual mesh filename=package://spider_bot/meshes/hip1_link.STL
- added link hip2_link, mass 0.020238; collision mesh filename=package://spider_bot/meshes/hip2_link.STL; visual mesh filename=package://spider_bot/meshes/hip2_link.STL
- added link hip3_link, mass 0.020238; collision mesh filename=package://spider_bot/meshes/hip3_link.STL; visual mesh filename=package://spider_bot/meshes/hip3_link.STL
- added link hip4_link, mass 0; collision mesh filename=package://spider_bot/meshes/hip4_link.STL; visual mesh filename=package://spider_bot/meshes/hip4_link.STL
- added link leg1_link, mass 0.0071825; collision mesh filename=package://spider_bot/meshes/leg1_link.STL; visual mesh filename=package://spider_bot/meshes/leg1_link.STL
- added link leg2_link, mass 0.0071825; collision mesh filename=package://spider_bot/meshes/leg2_link.STL; visual mesh filename=package://spider_bot/meshes/leg2_link.STL
- added link leg3_link, mass 0.0071825; collision mesh filename=package://spider_bot/meshes/leg3_link.STL; visual mesh filename=package://spider_bot/meshes/leg3_link.STL
- added link leg4_link, mass 0.0071825; collision mesh filename=package://spider_bot/meshes/leg4_link.STL; visual mesh filename=package://spider_bot/meshes/leg4_link.STL
- link base_link: mass 0.311250825006862 -> 0.31125
Joints:
- joint hip1: axis 0 1 0 -> 1 0 0; child hip1 -> hip1_link; origin xyz=0.1025 -0.065 0 rpy=1.5708 0 -2.815 -> xyz=0.1025 -0.065 0 rpy=1.2442 -1.5708 0
- joint hip2: child hip2 -> hip2_link
- joint hip3: child hip3 -> hip3_link
- joint hip4: child hip4 -> hip4_link; origin xyz=-0.1025 -0.065 0 rpy=1.5708 0 2.4418 -> xyz=-0.1025 -0.065 0 rpy=1.5708 0 2.4479
- joint leg1: child leg1 -> leg1_link; limit lower=-3.14 upper=3.14 effort=0 velocity=0 -> lower=-3.14 upper=3.14 effort=100 velocity=3; origin xyz=0 -0.01358 -0.01 rpy=-1.5708 -0.11409 1.5708 -> xyz=-0.01358 0 0.01 rpy=1.5708 0.11409 0; parent hip1 -> hip1_link
- joint leg2: child leg2 -> leg2_link; parent hip2 -> hip2_link
- joint leg3: child leg3 -> leg3_link; parent hip3 -> hip3_link
- joint leg4: child leg4 -> leg4_link; origin xyz=-0.025418 -0.01358 -0.01 rpy=-1.5708 -0.027408 1.5708 -> xyz=-0.028647 -0.01358 -0.01 rpy=-1.5708 -0.13243 1.5708; parent hip4 -> hip4_link
